File: MRBx60/MRBx60.kicad_pcb (KiCad board)
At the start: 2 copper layers, 300 x 200 mm, 185 parts, among them IC2 ICE40HX1K-TQ144, J1 Conn_02x35_Odd_Even, J10 Conn_01x04_Pin, J11 Conn_01x04_Pin, J12 Conn_01x04_Pin, J13 Conn_02x16_Odd_Even, J14 Conn_01x02_Pin, J15 Conn_01x02_Pin, J16 Conn_01x02_Pin, J17 Conn_01x02_Pin, J18 Conn_01x02_Pin, J19 Conn_02x12_Odd_Even, J2 Conn_02x35_Odd_Even, J20 Conn_02x12_Odd_Even, J21 Conn_02x08_Odd_Even, J22 Conn_02x08_Odd_Even, J23 Conn_02x08_Odd_Even, J24 Conn_02x08_Odd_Even, J25 Conn_02x08_Odd_Even, J26 Conn_02x08_Odd_Even, J27 Conn_02x08_Odd_Even, J28 Conn_02x16_Odd_Even, J29 Conn_02x16_Odd_Even, J3 Conn_01x02, J30 Conn_01x02, J31 Conn_02x16_Odd_Even, J4 Conn_01x08_Pin, J5 Conn_01x02_Pin, J6 USB_B, J7 Conn_01x02_Pin, J8 Conn_01x04_Socket, J9 Conn_01x05_Socket, SW0 SW_Reed_SPDT, SW1 SW_Reed_SPDT, SW10 SW_Reed_SPDT, SW11 SW_Reed_SPDT, SW12 SW_Reed_SPDT, SW13 SW_Reed_SPDT, SW14 SW_Reed_SPDT, SW15 SW_Reed_SPDT, SW16 SW_Reed_SPDT, SW17 SW_Reed_SPDT, SW2 SW_Reed_SPDT, SW20 SW_Push_Dual_x2, SW21 SW_Push_Dual_x2, SW3 SW_Reed_SPDT, SW4 SW_Push_Dual_x2, SW5 SW_Push_Dual_x2, U1 FT2232HL, U10 93AAxxA, U11 BME280, U12 ADS1115IDGS, U13 PC817, U14 PC817, U15 PC817, U16 PC817, U17 PC817, U18 PC817, U19 PC817, U2 PC817, U20 PC817, U21 PC817, U22 PC817, U23 PC817, U24 PC817, U25 PC817, U26 PC817, U27 PC817, U28 PC817, U29 PC817, U3 L7812, U30 PC817, U31 PC817, U32 PC817, U33 PC817, U34 PC817, U35 PC817, U36 ADS1115IDGS, U4 L7805, U5 L7824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

Commit message: Add files via upload
dodawanie ścieżek, podejscie 1
Parts:
- J13: moved to B.Cu
- moved R35 135.8 mm to (262.9, 388.6)
- moved R47 108.7 mm to (135.6, 389.4)
- moved R49 97.0 mm to (122.4, 379.0)
- moved R36 95.7 mm to (276.1, 379.0)
- moved R48 83.9 mm to (148.3, 379.0)
- moved R37 82.9 mm to (250.4, 379.0)
- moved R38 73.5 mm to (276.1, 388.6)
- moved R26 71.9 mm to (184.4, 388.9)
- moved R13 69.0 mm to (184.7, 379.0)
- moved U2 61.4 mm to (174.0, 373.4)
- moved R45 57.7 mm to (212.1, 388.6)
- moved U34 52.7 mm to (112.0, 381.8)
- moved U18 51.8 mm to (252.7, 382.3)
- moved R51 51.3 mm to (122.4, 389.1)
- moved U35 51.3 mm to (125.2, 373.4)
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Connections:
- J31 pad 1: IOL_12B -> unconnected-(J31-Pin_1-Pad1)
- J31 pad 13: unconnected-(J31-Pin_13-Pad13) -> IOR_60
- J31 pad 15: unconnected-(J31-Pin_15-Pad15) -> IOR_61
- J31 pad 3: IOL_12A -> unconnected-(J31-Pin_3-Pad3)
- J31 pad 5: IOL_11B -> unconnected-(J31-Pin_5-Pad5)
- J31 pad 7: IOL_11A -> unconnected-(J31-Pin_7-Pad7)
Routing:
- net PD_0: track 0.00 -> 219.9 mm, vias 0 -> 1
- net PD_1: track 0.00 -> 219.6 mm, vias 0 -> 2
- net IOB_25: track 0.00 -> 187.5 mm, vias 0 -> 2
- net PB_7: track 0.00 -> 175.5 mm, vias 0 -> 3
- net PG_12: track 0.00 -> 175.1 mm, vias 0 -> 1
- net IOR_62: track 0.00 -> 168.7 mm
- net PD_7: track 0.00 -> 166.6 mm, vias 0 -> 3
- net PD_6: track 0.00 -> 165.2 mm, vias 0 -> 2
- net PD_5: track 0.00 -> 161.8 mm, vias 0 -> 3
- net PD_4: track 0.00 -> 158.4 mm, vias 0 -> 3
- net IOR_65: track 0.00 -> 157.9 mm
- net IOR_63: track 0.00 -> 156.3 mm
- net IOR_57: track 0.00 -> 156.1 mm, vias 0 -> 2
- net IOR_64: track 0.00 -> 154.6 mm
- net PF_7: track 0.00 -> 145.5 mm, vias 0 -> 3
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- removed copper zone on F.Cu, net GND
Other:
- board text added: "Ext PWR"
- board text added: "gnd"
- board text added: "supply"
- board text removed: "FPGA"
- board text removed: "Programmer"
- board text removed: "STM"
- board text removed: "STM Dock station"
