File: SimpleLattice/PWR.kicad_sch (KiCad schematic)
At the start: 5 parts, among them J12 Conn_01x16_Pin, J14 USB_B, J15 Conn_01x02_Pin, J16 Conn_01x02_Pin, U7 LD1117S50TR_SOT223

Commit message: Add files via upload
kolejne polaczenia v2
Parts:
- U7: footprint Package_TO_SOT_SMD:SOT-223-3_TabPin2 -> Package_TO_SOT_THT:TO-220-3_Vertical
Changed lines of the file:
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@@
       (effects (font (size 1.27 1.27)))
     )
-    (property "Footprint" "Package_TO_SOT_SMD:SOT-223-3_TabPin2" (at 106.68 49.53 0)
+    (property "Footprint" "Package_TO_SOT_THT:TO-220-3_Vertical" (at 106.68 49.53 0)
       (effects (font (size 1.27 1.27)) hide)
     )
