File: SimpleLattice/STM_dock.kicad_sch (KiCad schematic)
At the start: 2 parts, among them J4 Conn_02x19_Odd_Even, J5 Conn_02x19_Odd_Even

Commit message: Add files via upload
kolejne polaczenia v2
Connections:
- net PC7: now also J5.19 (Pin_19)
Changed lines of the file:
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@@
     )
   )
-  (global_label "PC7" (shape bidirectional) (at 101.6 52.07 180) (fields_autoplaced)
+  (global_label "PC7" (shape bidirectional) (at 101.6 52.705 180) (fields_autoplaced)
     (effects (font (size 1.27 1.27)) (justify right))
-    (property "Intersheetrefs" "${INTERSHEET_REFS}" (at 93.8334 52.07 0)
+    (property "Intersheetrefs" "${INTERSHEET_REFS}" (at 93.8334 52.705 0)
       (effects (font (size 1.27 1.27)) (justify right) hide)
     )
