File: SimpleLattice/SimpleLattice.kicad_sch (KiCad schematic)
At the start: 19 parts, among them IC1 LCMXO2-1200ZE-1TG144C, J1 Conn_01x08_Pin, J10 Conn_01x16_Pin, J11 Conn_01x16_Pin, J12 Conn_01x16_Pin, J2 Conn_01x08_Pin, J3 Conn_01x10_Pin, J9 Conn_01x16_Pin, Y1 CB3LV-3C-50M0000

Commit message: Add files via upload
kolejne polaczenia v2
Parts:
- removed J12: Conn_01x16_Pin, Connector_PinHeader_1.27mm:PinHeader_1x16_P1.27mm_Vertical, symbol Connector:Conn_01x16_Pin
