File: SimpleLattice/SimpleLattice.kicad_pcb (KiCad board)
At the start: 2 copper layers, 160 x 120 mm, 67 parts, among them IC1 LCMXO2-1200ZE-1TG144C, J1 Conn_01x08_Pin, J10 Conn_01x16_Pin, J11 Conn_01x16_Pin, J2 Conn_01x08_Pin, J3 Conn_01x10_Pin, J4 Conn_02x19_Odd_Even, J5 Conn_02x19_Odd_Even, J6 Conn_01x02, J7 Conn_01x02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

Commit message: Add files via upload
kolejne polaczenia v2
Parts:
- added J13: Conn_01x16_Pin, Connector_PinHeader_1.27mm:PinHeader_1x16_P1.27mm_Vertical, F.Cu at (174.0, 34.0)
- added J14: USB_B, Connector_USB:USB_B_Amphenol_MUSB-D511_Vertical_Rugged, F.Cu at (203.5, 41.2)
- added J15: Conn_01x02_Pin, Connector_PinHeader_1.27mm:PinHeader_1x02_P1.27mm_Vertical, F.Cu at (185.5, 35.9)
- added J16: Conn_01x02_Pin, Connector_PinHeader_1.27mm:PinHeader_1x02_P1.27mm_Vertical, F.Cu at (179.6, 35.9)
- added U7: LD1117S50TR_SOT223, Package_TO_SOT_THT:TO-220-3_Vertical, F.Cu at (179.9, 49.0)
- moved U1 87.9 mm to (56.4, 119.4)
- moved R21 87.8 mm to (48.9, 115.0)
- moved R31 80.3 mm to (130.9, 115.0)
- moved U6 80.2 mm to (137.3, 119.2)
- moved R23 54.0 mm to (64.9, 115.0)
- moved U2 54.0 mm to (72.2, 119.4)
- moved R29 47.1 mm to (114.9, 115.0)
- moved U5 47.1 mm to (122.0, 119.3)
- moved R25 20.9 mm to (80.9, 115.0)
- moved U3 20.9 mm to (88.5, 119.3)
- moved J4 19.8 mm to (212.7, 67.5)
- moved J5 19.8 mm to (212.7, 129.7)
- moved C3 14.8 mm to (111.0, 70.0)
- moved C1 13.0 mm to (123.4, 100.2)
- moved R27 12.8 mm to (97.9, 115.0)
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Connections:
- IC1 pad 82: unconnected-(IC1-PR9A-Pad82) -> Net-(IC1-PR9A)
- J5 pad 19: unconnected-(J5-Pin_19-Pad19) -> PC7
- J9 pad 15: unconnected-(J9-Pin_15-Pad15) -> Net-(IC1-PR9A)
- J9 pad 16: unconnected-(J9-Pin_16-Pad16) -> GND
Routing:
- net PC9: track 0.00 -> 145.0 mm, vias 0 -> 2
- net PC8: track 0.00 -> 141.0 mm, vias 0 -> 2
- net PC6: track 0.00 -> 139.6 mm, vias 0 -> 2
- net PC5: track 0.00 -> 137.3 mm, vias 0 -> 2
- net PB2: track 0.00 -> 125.6 mm, vias 0 -> 2
- net PB12: track 0.00 -> 121.0 mm, vias 0 -> 2
- net PB1: track 0.00 -> 120.2 mm, vias 0 -> 2
- net PB15: track 0.00 -> 113.1 mm, vias 0 -> 2
- net PB14: track 0.00 -> 109.3 mm, vias 0 -> 2
- net PB13: track 0.00 -> 108.1 mm, vias 0 -> 2
- net PC10: track 0.00 -> 105.7 mm, vias 0 -> 1
- net PC4: track 0.00 -> 102.3 mm, vias 0 -> 2
- net PC7: track 0.00 -> 101.8 mm, vias 0 -> 3
- net PC11: track 0.00 -> 97.1 mm, vias 0 -> 1
- net LED7: track 0.00 -> 94.4 mm
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Other:
- board size 160 x 120 mm -> 180 x 120 mm

Commit message: Add files via upload
kolejnme p-olaczenia prawie koniec
Parts:
- J8: moved to B.Cu
- moved R2 11.0 mm to (70.9, 100.8), turned to 180 degrees
- moved R3 11.0 mm to (70.9, 97.0), turned to 180 degrees
- moved R1 10.2 mm to (70.8, 92.9), turned to 180 degrees
- moved J8 7.15 mm to (59.5, 141.4)
- moved R6 2.38 mm to (90.6, 96.0)
- moved R5 2.38 mm to (90.6, 87.9)
Routing:
- net 3V3: track 7.30 -> 213.6 mm, vias 1 -> 4
- net Ext_GND: track 0.00 -> 114.2 mm
- net TMS: track 0.00 -> 112.0 mm, vias 0 -> 1
- net TDI: track 0.00 -> 108.1 mm, vias 0 -> 1
- net TCK: track 0.00 -> 107.3 mm, vias 0 -> 1
- net TDO: track 0.00 -> 105.3 mm, vias 0 -> 1
- net OUT5: track 0.00 -> 99.5 mm
- net OUT6: track 0.00 -> 79.1 mm
- net OUT4: track 0.00 -> 73.4 mm
- net ADC_SDA: track 72.1 -> 0.00 mm
- net ADC_SCL: track 72.0 -> 0.00 mm
- net Net-(J3-Pin_5): track 0.00 -> 70.1 mm
- net OUT1: track 0.00 -> 67.4 mm
- net OUT2: track 0.00 -> 60.0 mm, vias 0 -> 2
- net Net-(IC1-PR9A): track 0.00 -> 59.8 mm
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
Commit message: Add files via upload
Routing:
- net 3V3: track 213.6 -> 433.9 mm, vias 4 -> 13
- net ADC_SCL: track 0.00 -> 106.4 mm, vias 0 -> 2
- net ADC_ALERT: track 0.00 -> 105.6 mm, vias 0 -> 2
- net ADC_SDA: track 0.00 -> 102.4 mm, vias 0 -> 2
- net Ext_VCC: track 55.6 -> 131.4 mm
- net GND: track 0.00 -> 55.3 mm, vias 0 -> 10
- net KEY1: track 80.2 -> 86.7 mm
- net KEY0: track 72.5 -> 79.0 mm
- net J11_12: track 55.5 -> 56.2 mm
- net CLK: track 29.0 -> 29.5 mm
Other:
- board text added: "3v3"
- board text added: "ADC"
- board text added: "D+ D-"
- board text added: "GND"
- board text added: "GND 9A 8D 8C 8B 8A 5D 5C 5B 5A 4D 4C 4B 4A 3B 3A"
- board text added: "J pwr"
- board text added: "JTAG"
- board text added: "MRBx10"
- board text added: "Optic Output"
- board text added: "PC10"
- board text added: "PC8"
- board text added: "PC9"
- board text added: "Rx Tx RTSn CTSn DTRn DSRn DCDn"
- board text added: "RxTx"
- board text added: "STM docking"
- board text added: "SW"
